Commit message: huge variations in launch files of gazebo simulations

File: shelfino_description/models/shelfino/model.sdf.xacro (robot description, xacro)
@@ -1,8 +1,10 @@
 <?xml version='1.0'?>
-<sdf version='1.4'>
+<sdf version='1.4' xmlns:xacro="http://www.ros.org/wiki/xacro">
+  <xacro:arg name="robot_id" default="X" />
+  <xacro:macro name="shelfino" params="robot_id">
 <!--
                                                       SHELFINO MODEL
 -->
-  <model name="shelfino">
+  <model name="shelfino${robot_id}">
 <!--
                                                       BODY OF SHELFINO
@@ -222,9 +224,9 @@
           <ros>
             <!-- Set namespace -->
-            <!-- <namespace>${robot_name}</namespace> -->
+            <!-- <namespace>${robot_id}</namespace> -->
             <remapping>~/out:=scan</remapping>
           </ros>
           <output_type>sensor_msgs/LaserScan</output_type>
-          <frame_name>base_laser</frame_name>
+          <frame_name>shelfino${robot_id}/base_laser</frame_name>
         </plugin>
       </sensor>
@@ -234,9 +236,9 @@
 -->
     <plugin name="differential_drive_controller" filename="libgazebo_ros_diff_drive.so">
-      <ros>
+      <!-- <ros> -->
         <!-- Set namespace -->
-        <!-- <namespace>${robot_name}</namespace> -->
-        <remapping>/tf:=tf</remapping>
-      </ros>
+        <!-- <namespace>${robot_id}</namespace> -->
+        <!-- <remapping>/tf:=tf</remapping> -->
+      <!-- </ros> -->
       <!-- <alwaysOn>true</alwaysOn> -->
       <update_rate>30</update_rate>
@@ -256,6 +258,6 @@
       <publish_odom_tf>true</publish_odom_tf>
       <publish_wheel_tf>false</publish_wheel_tf>
-      <odometry_frame>odom</odometry_frame>
-      <robot_base_frame>base_link</robot_base_frame>
+      <odometry_frame>shelfino${robot_id}/odom</odometry_frame>
+      <robot_base_frame>shelfino${robot_id}/base_link</robot_base_frame>
       <!-- <odometrySource>ENCODER</odometrySource> -->
       <!-- <odometrySource>WORLD</odometrySource> -->
@@ -273,3 +275,5 @@
     </plugin>
   </model>
+  </xacro:macro>
+  <xacro:shelfino robot_id="$(arg robot_id)" />
 </sdf>

File: shelfino_description/models/shelfino/model.urdf.xacro (robot description, xacro)
@@ -1,4 +1,6 @@
-<?xml version='1.0'?>
-<robot name="shelfino">
+<?xml version='1.0' ?>
+<robot name="shelfino" xmlns:xacro="http://www.ros.org/wiki/xacro">
+  <xacro:arg name="robot_id" default="X" />
+  <xacro:macro name="shelfino" params="robot_id">
   <!--
                                                         MATERIALS
@@ -16,5 +18,5 @@
                                                         BODY OF SHELFINO
   -->
-    <link name='base_link'>
+    <link name='shelfino${robot_id}/base_link'>
       <visual name='body_visual'>
         <origin xyz='0 0 0.25'/>
@@ -49,6 +51,6 @@
   -->
     <joint name="wheel_left_joint" type="continuous">
-      <parent link="base_link"/>
-      <child link="left_wheel"/>
+      <parent link="shelfino${robot_id}/base_link"/>
+      <child link="shelfino${robot_id}/left_wheel"/>
       <origin xyz="0 0.27 0.125" rpy="0 1.5707 1.5707"/>
       <axis xyz="0 0 1"/>
@@ -57,5 +59,5 @@
                                                         LEFT WHEEL
   -->
-    <link name="left_wheel">
+    <link name="shelfino${robot_id}/left_wheel">
       <visual name="visual">
         <geometry>
@@ -80,6 +82,6 @@
   -->
     <joint name="wheel_right_joint" type="continuous">
-      <parent link="base_link"/>
-      <child link="right_wheel"/>
+      <parent link="shelfino${robot_id}/base_link"/>
+      <child link="shelfino${robot_id}/right_wheel"/>
       <origin xyz="0 -0.27 0.125" rpy="0 1.5707 1.5707"/>
       <axis xyz="0 0 1"/>
@@ -88,5 +90,5 @@
                                                         RIGHT WHEEL
   -->
-    <link name="right_wheel">
+    <link name="shelfino${robot_id}/right_wheel">
       <visual name="visual">
         <geometry>
@@ -111,6 +113,6 @@
   -->
     <joint name="lidar2d_joint" type="fixed">
-      <parent link="base_link"></parent>
-      <child link="base_laser"></child>
+      <parent link="shelfino${robot_id}/base_link"></parent>
+      <child link="shelfino${robot_id}/base_laser"></child>
       <origin xyz="0 0 0.45" rpy="0 0 0"/>
     </joint>
@@ -118,5 +120,5 @@
                                                         LIDAR
   -->
-    <link name="base_laser">
+    <link name="shelfino${robot_id}/base_laser">
       <visual>
         <geometry>
@@ -139,3 +141,5 @@
       </inertial>
     </link>
+  </xacro:macro>
+  <xacro:shelfino robot_id="$(arg robot_id)" />
 </robot>
